Commit message: updata virtual joints and add claw meshes

File: urdf/ebamk2_mesh.urdf (robot description, URDF)
Before this commit: robot ebamk2, 7 links, 6 joints
Links:
- added link claw_l; visual mesh filename=package://ebamk2_description/meshes/claw_l.STL scale=0.001 0.001 0.001
- added link claw_r; visual mesh filename=package://ebamk2_description/meshes/claw_r.STL scale=0.001 0.001 0.001
- link claw_base: geometry visual mesh filename=package://ebamk2_description/meshes/link_5.STL scale=0.001 0.001 0.001
- link link_2v: geometry collision cylinder length=0.0001 radius=0.0001; visual cylinder length=0.001 radius=0.05
- link link_4: geometry visual mesh filename=package://ebamk2_description/meshes/link_4.STL scale=0.001 0.001 0.001
Joints:
- added joint joint_6: type revolute, parent claw_base, child claw_l, origin xyz=0.0196 0.021 -0.004 rpy=0 0 0, axis 0 0 1, limit lower=-0.15 upper=0.65 effort=0 velocity=1.0
- added joint joint_7: type revolute, parent claw_base, child claw_r, origin xyz=0.0196 0.0040 -0.004 rpy=0 0 0, axis 0 0 -1, limit lower=-0.15 upper=0.65 effort=0 velocity=1.0, mimic joint=joint_6 multiplier=1.0 offset=0
- joint joint_2: limit lower=-0.6109 upper=0.9599 effort=0 velocity=0 -> lower=-0.80 upper=0.35 effort=0 velocity=0
- joint joint_3: limit lower=-1.2217 upper=0.3491 effort=0 velocity=0 -> lower=-0.70 upper=0.50 effort=0 velocity=0
- joint joint_4: axis 0 0 1 -> 0 1 0; mimic (none) -> joint=joint_3 multiplier=1 offset=0; origin xyz=0.147 0 0 rpy=0 0 0 -> xyz=0.1459 0.0185 0.0203 rpy=0 1.570796325 3.14159
- joint joint_5: origin xyz=0.04 0 0.002 rpy=0 0 0 -> xyz=-0.0095 0.001 -0.033 rpy=-0 1.570796325 0

Commit message: cosmetic changes on urdf

File: urdf/ebamk2_mesh.urdf (robot description, URDF)
Before this commit: robot ebamk2, 9 links, 8 joints
Joints:
- joint joint_6: limit lower=-0.15 upper=0.65 effort=0 velocity=1.0 -> lower=0 upper=0.65 effort=0 velocity=1.0
- joint joint_7: limit lower=-0.15 upper=0.65 effort=0 velocity=1.0 -> lower=0 upper=0.65 effort=0 velocity=1.0
