Commit message: add mimic virtual joints to urdf

File: urdf/ebamk2.urdf (robot description, URDF)
Before this commit: robot ebamk2, 8 links, 7 joints
Links:
- added link link_2v; collision cylinder length=0.001 radius=0.01; visual cylinder length=0.001 radius=0.01
- link claw_l: geometry visual box size=0.005 0.047 0.005
- link claw_r: geometry visual box size=0.005 0.047 0.005
Joints:
- removed joint joint6
- removed joint joint7
- added joint joint2v: type revolute, parent link_2, child link_2v, origin xyz=0 0 0.135 rpy=0 0 0, axis 1 0 0, limit lower=1.00 upper=1.00 effort=30 velocity=1.0, mimic joint=joint_2 multiplier=-1 offset=0
- added joint joint_6: type revolute, parent claw_base, child claw_l, origin xyz=-0.01 0.01 0 rpy=0 0 0, axis 0 0 1, limit lower=-0.15 upper=0.65 effort=1.0 velocity=1.0
- added joint joint_7: type revolute, parent claw_base, child claw_r, origin xyz=0.01 0.01 0 rpy=0 0 0, axis 0 0 -1, limit lower=-0.15 upper=0.65 effort=1.0 velocity=1.0, mimic joint=joint_6 multiplier=1.0 offset=0
- joint joint_2: limit lower=-0.6109 upper=0.9599 effort=0 velocity=0 -> lower=-1.0 upper=0.65 effort=0 velocity=0
- joint joint_3: limit lower=-1.2217 upper=0.3491 effort=0 velocity=0 -> lower=-0.90 upper=0.20 effort=0 velocity=0; origin xyz=0 0 0.135 rpy=0 0 0 -> xyz=0 0 0 rpy=0 0 0; parent link_2 -> link_2v
- joint joint_4: mimic (none) -> joint=joint_3 multiplier=-1 offset=0

File: urdf/ebamk2_mesh.urdf (robot description, URDF)
Before this commit: robot ebamk2, 6 links, 5 joints
Links:
- added link link_2v; collision cylinder length=0.001 radius=0.01; visual cylinder length=0.001 radius=0.05
Joints:
- added joint joint2v: type revolute, parent link_2, child link_2v, origin xyz=-0.021 0.135 -0.0105 rpy=1.570796325 0 0, axis 0 1 0, limit lower=1.570796325 upper=1.570796325 effort=30 velocity=1.0, mimic joint=joint_2 multiplier=-1 offset=0
- joint joint_2: origin xyz=0 -0.005 0.035 rpy=1.578 0 0 -> xyz=0 -0.005 0.037 rpy=1.578 0 0
- joint joint_3: axis 0 0 1 -> 0 1 0; origin xyz=-0.021 0.133 -0.0105 rpy=0 0 0 -> xyz=0 0 0 rpy=0 0 0; parent link_2 -> link_2v

Commit message: change to mimic joint limits

File: urdf/ebamk2.urdf (robot description, URDF)
Before this commit: robot ebamk2, 9 links, 8 joints
Links:
- link link_2v: geometry collision cylinder length=0.001 radius=0.001; visual cylinder length=0.001 radius=0.001
Joints:
- joint joint2v: limit lower=1.00 upper=1.00 effort=30 velocity=1.0 -> lower=-3.14159 upper=3.14159 effort=30 velocity=1.0

File: urdf/ebamk2_mesh.urdf (robot description, URDF)
Before this commit: robot ebamk2, 9 links, 8 joints
Links:
- link link_2v: geometry collision cylinder length=0.0001 radius=0.0001; visual cylinder length=0.001 radius=0.0001
Joints:
- joint joint2v: limit lower=1.570796325 upper=1.570796325 effort=30 velocity=1.0 -> lower=-3.14159 upper=3.14159 effort=30 velocity=1.0
- joint joint_4: limit lower=-1.01 upper=1.01 effort=0 velocity=0 -> lower=-3.14159 upper=3.14159 effort=0 velocity=0

Commit message: Cleanup and minor changes

File: urdf/ebamk2.urdf (robot description, URDF)
Before this commit: robot ebamk2, 9 links, 8 joints
Joints:
- joint joint_2: limit lower=-1.0 upper=0.65 effort=0 velocity=0 -> lower=-0.80 upper=0.35 effort=0 velocity=0
- joint joint_3: limit lower=-0.90 upper=0.20 effort=0 velocity=0 -> lower=-0.77 upper=0.45 effort=0 velocity=0

File: urdf/ebamk2_mesh.urdf (robot description, URDF)
Before this commit: robot ebamk2, 9 links, 8 joints
Links:
- link base_link: geometry collision cylinder length=0.0001 radius=0.0001; visual mesh filename=package://ebamk2_description/meshes/base_link.STL
Joints:
- joint joint_3: limit lower=-0.70 upper=0.50 effort=0 velocity=0 -> lower=-0.77 upper=0.45 effort=0 velocity=0
