Commit message: ebamk2_mesh updade and new urdf files

File: urdf/ebamk2_mesh_all_mimic.urdf (robot description, URDF)
Before this commit: robot ebamk2, 9 links, 8 joints
Joints:
- joint joint_4: mimic (none) -> joint=joint_3 multiplier=1 offset=0

File: urdf/ebamk2_mesh_no_mimic.urdf (robot description, URDF)
Before this commit: robot ebamk2, 9 links, 8 joints
Links:
- removed link link_2v
Joints:
- removed joint joint2v
- joint joint_3: axis 0 1 0 -> 0 0 1; origin xyz=0 0 0 rpy=0 0 0 -> xyz=-0.021 0.133 -0.0105 rpy=0 0 0; parent link_2v -> link_2
- joint joint_4: origin xyz=0.1459 0.0185 0.0203 rpy=0 1.570796325 3.14159 -> xyz=0.147 0 0.018 rpy=-1.570796325 0 1.570796325
